File: schematic/betterstarbie.kicad_sch (KiCad schematic)
At the start: 7 parts, among them J1 Conn_01x04_Pin, J2 Conn_01x08_Pin, SW1 SW_Push, SW2 SW_Push, U1 DHT11, U2 XIAO-ESP32-C3-SMD

Commit message: Add files via upload
Parts:
- removed J2: Conn_01x08_Pin, Connector_PinHeader_2.54mm:PinHeader_1x08_P2.54mm_Vertical, symbol Connector:Conn_01x08_Pin
- removed R1: 10k, Resistor_THT:R_Axial_DIN0204_L3.6mm_D1.6mm_P7.62mm_Horizontal, symbol Device:R
- removed U1: DHT11, Sensor:Aosong_DHT11_5.5x12.0_P2.54mm, symbol Sensor:DHT11
- added C0, C1, C2, C3, C4, C5: 100nF, Capacitor_SMD:C_0603_1608Metric, symbol Device:C
- added D1, D2, D3, D4, D5: WS2812B-2020, LED_SMD:LED_WS2812B-2020_PLCC4_2.0x2.0mm, symbol LED:WS2812B-2020
- added J2, J3: Conn_01x02_Socket, Connector_PinSocket_2.54mm:PinSocket_1x02_P2.54mm_Vertical, symbol Connector:Conn_01x02_Socket
- added J4, J5: Conn_01x02_Pin, Connector_PinHeader_2.54mm:PinHeader_1x02_P2.54mm_Horizontal, symbol Connector:Conn_01x02_Pin
- added J6: ENS160+AHT21, Connector_PinSocket_2.54mm:PinSocket_1x08_P2.54mm_Vertical, symbol Connector:Conn_01x08_Socket
- added J7: HLK-LD2450 2x4 2.00mm, Connector_PinSocket_2.00mm:PinSocket_2x04_P2.00mm_Vertical, symbol Connector_Generic:Conn_02x04_Odd_Even
- added R3: 330Ω, Resistor_SMD:R_0603_1608Metric, symbol Device:R
- added U3: 74AHCT1G125, Package_TO_SOT_SMD:SOT-23-5, symbol 74xGxx:74AHCT1G125
- J1: value Conn_01x04_Pin -> OLED_SH1107_1.5in; footprint Imported Parts:Display_128x64_096_I2C -> Connector_PinSocket_2.54mm:PinSocket_1x04_P2.54mm_Vertical; symbol Connector:Conn_01x04_Pin -> Connector:Conn_01x04_Socket
- U2: value XIAO-ESP32-C3-SMD -> XIAO-ESP32-S3-SMD; footprint Imported Parts:XIAO-ESP32-C6-DIP -> Seed Studio Library for Kicad:XIAO-ESP32-S3-DIP
Connections:
- net +3.3V: now also J6.1 (Pin_1); no longer J1.2 (Pin_2)
- net +5V: now also J1.1 (Pin_1), C0.1, C1.1, C2.1, C3.1, C4.1, C5.2, J7.2 (Pin_2), U3.5 (VCC)
- net GND: now also J1.2 (Pin_2), C5.1, D1.2 (VSS), D2.2 (VSS), D3.2 (VSS), D4.2 (VSS), D5.2 (VSS), J2.2 (Pin_2), J3.2 (Pin_2), J6.3 (Pin_3), J6.6 (Pin_6), J6.7 (Pin_7), J7.8 (Pin_8), U3.1, U3.3 (GND); no longer J1.1 (Pin_1), SW1.2, SW2.2
- net SCL: now also J6.4 (Pin_4)
- net SDA: now also J6.5 (Pin_5)
- net RADAR_TX: now reaches U2.7 (D6)
- net RADAR_TX: now also J7.3 (Pin_3)
- net RADAR_RX: now reaches U2.8 (D7)
- net RADAR_RX: now also J7.1 (Pin_1)
- net DHT11 DATA renamed BTN1
- net BTN1: now also J2.1 (Pin_1)
- net GPIO2: no longer names the net of SW1.1
- net GPIO2: now also J4.2 (Pin_2); no longer U2.3 (D2)
- net GPIO3: no longer names the net of SW2.1
- net GPIO3: now also J5.2 (Pin_2); no longer U2.4 (D3)
- new net: R3.1, U3.4
- new net: C2.2, D3.4 (VDD)
- new net: J5.1 (Pin_1), SW2.2
- new net: C4.2, D5.4 (VDD)
- new net: D1.1 (DOUT), D2.3 (DIN)
- new net: D1.3 (DIN), R3.2
- new net: C0.2, D1.4 (VDD)
- new net: J4.1 (Pin_1), SW1.2
- new net: C1.2, D2.4 (VDD)
- new net: D3.1 (DOUT), D4.3 (DIN)
- new net: D2.1 (DOUT), D3.3 (DIN)
- new net: D4.1 (DOUT), D5.3 (DIN)
- new net: C3.2, D4.4 (VDD)
- new net BTN2: J3.1 (Pin_1), U2.3 (D2)
- new net LED Data: U2.4 (D3), U3.2
- no-connect marks 17 -> 18
Other:
- note added: "3V3 (output?)"
- note added: "5 Leds WS2812B"
- note added: "ADD"
- note added: "Buttons (Daughter Board)"
- note added: "Buttons Connector"
- note added: "CS"
- note added: "Environment sensor ENS160+AHT21 (air quality + temp + humidity)"
- note added: "GND"
- note added: "INT"
- note added: "MMWave sensor HLK-LD2450"
- note added: "OLED SCREEN 1.5in SH1107 128x128"
- note added: "SCL"
- note added: "SDA"
- note added: "VCC"
- note added: "VIN"
- note added: "XIAO Seedstudio ESP32S3"
- note removed: "Buttons!"
- note removed: "Enviroment sensor (temp and humidity)"
- note removed: "MPU6050"
- note removed: "OLED SCREEN"
- note removed: "XIAO Seedstudio ESP32 C3"
- title: Better Starbie -> R-Bot
- moved on the sheet: SW1, SW2, U2
